File: hw/adbuino_v0p9/adbuino.sch (KiCad schematic (older format))
At the start: 25 parts, among them IC1 MAX3421EEHJ+, J1 U254-051N-4BH806, J2 USB_A, J3 Mini-DIN-4, J4 Mini-DIN-4, SW1 SW_Push, U1 ATmega328P-AU, U2 AMS1117-3.3

Commit message: Finished initial board layout
Parts:
- added C10, C11: 30p, Capacitor_SMD:C_0805_2012Metric, symbol Device:C_Small
- added C12, C13, C14, C15, C16, C2, C5: 100n, Capacitor_SMD:C_0805_2012Metric, symbol Device:C_Small
- added C6, C7: 4p, Capacitor_SMD:C_0805_2012Metric, symbol Device:C_Small
- added F1: Polyfuse, Fuse:Fuse_0805_2012Metric_Castellated, symbol Device:Polyfuse
- added IC2: 74HC4050D,653, Package_SO:SOP-16_3.9x9.9mm_P1.27mm, symbol SamacSys_Parts:74HC4050D,653
- added JP2: SolderJumper_3_Bridged12, Jumper:SolderJumper-3_P1.3mm_Bridged12_RoundedPad1.0x1.5mm_NumberLabels, symbol Jumper:SolderJumper_3_Bridged12
- added JP3, JP4, JP5, JP6: SolderJumper_2_Bridged, Jumper:SolderJumper-2_P1.3mm_Bridged_RoundedPad1.0x1.5mm, symbol Jumper:SolderJumper_2_Bridged
- added R1: 1M, Resistor_SMD:R_0805_2012Metric, symbol Device:R_Small
- added R2: 10k, Resistor_SMD:R_0805_2012Metric, symbol Device:R_Small
- added SW1: SW_Push, Button_Switch_SMD:SW_Push_1P1T_NO_6x6mm_H9.5mm, symbol Switch:SW_Push
- added TP1, TP10, TP11, TP12, TP13, TP14, TP15, TP16, TP17, TP2, TP3, TP4, TP5, TP6, TP7, TP8, TP9: TestPoint_Small, TestPoint:TestPoint_Pad_D1.0mm, symbol Connector:TestPoint_Small
- added Y1: 16MHz, Crystal:Crystal_SMD_3225-4Pin_3.2x2.5mm, symbol Device:Crystal_GND24_Small
- added Y2: 12MHz, Crystal:Crystal_SMD_HC49-SD, symbol Device:Crystal_Small
- J1: renamed from J?; footprint (none) -> Connector_PinHeader_2.54mm:PinHeader_1x06_P2.54mm_Vertical
- JP1: renamed from JP?; footprint (none) -> Jumper:SolderJumper-3_P1.3mm_Bridged12_RoundedPad1.0x1.5mm_NumberLabels
- SW2: renamed from SW1; footprint Button_Switch_THT:SW_PUSH_6mm -> Button_Switch_SMD:SW_Push_1P1T_NO_6x6mm_H9.5mm; LCSC (none) -> C720316
- gave numbers to parts that had none: 1
- renumbered C3 to C1, C4 to C3, C5 to C4, C1 to C8, C2 to C9, J1 to J2, J2 to J3, J3 to J4, J4 to J5, JP1 to JP7, R1 to R4, R2 to R5, R3 to R6, R4 to R7, TP9 to TP18, TP10 to TP19, TP11 to TP20, TP12 to TP21, U2 to U1, U1 to U2
Connections:
- net +3V3: now also C13.2, IC2.1 (VCC), JP2.1 (A), R2.1; no longer U2.18 (AVCC), U2.4 (VCC), U2.6 (VCC)
- net FTDI_DTR: now also C5.2
- net GND: now also C10.2, C11.2, C12.2, C13.1, C14.2, C15.2, C16.2, C2.2, C6.2, C7.2, IC2.8 (GND), SW1.2, Y1.2, Y1.4
- net MAX3421_GPX: now also U2.12 (PB0), TP3.1
- net MAX3421_INT: now also U2.13 (PB1), TP4.1
- net MAX3421_RESET: now also IC2.10 (4Y), JP3.1 (A); no longer U2.11 (PD7)
- net MAX3421_SS: now also IC2.4 (2Y), JP5.1 (A); no longer U2.14 (PB2)
- net SPI_MISO: now also TP7.1
- net SPI_MOSI: now also IC2.6 (3Y), JP6.1 (A); no longer U2.15 (PB3)
- net SPI_SCLK: now also IC2.2 (1Y), JP4.1 (A); no longer U2.17 (PB5)
- net VBUS: now also F1.2, JP2.3 (B); no longer J3.1 (VBUS)
- net at IC1.22 (VBCOMP): now also C12.1
- net at IC1.24 (XI): now also C11.1, Y2.1
- net at IC1.25 (XO): now also C10.1, Y2.2
- net ADB_DATA_LV: now reaches U2.1 (PD3)
- net at U2.10 (PD6): now also TP17.1
- net at U2.19 (ADC6): now also TP1.1
- net at U2.2 (PD4): now also TP15.1
- net at U2.20 (AREF): now also C2.1
- net at U2.22 (ADC7): now also TP2.1
- net at U2.23 (PC0): now also TP9.1
- net at U2.24 (PC1): now also TP10.1
- net at U2.25 (PC2): now also TP11.1
- net at U2.26 (PC3): now also TP12.1
- net at U2.27 (PC4): now also TP13.1
- net at U2.28 (PC5): now also TP14.1
- net at U2.29 (~RESET~/PC6): now also C5.1, R2.2, SW1.1
- net ADB_PWR_ON_LV: now reaches U2.32 (PD2)
- net at U2.7 (XTAL1/PB6): now also C6.1, R1.1, Y1.3
- net at U2.8 (XTAL2/PB7): now also C7.1, R1.2, Y1.1
- net at U2.9 (PD5): now also TP16.1
- new net: F1.1, J3.1 (VBUS)
- new net TTL_MAX3421_RESET: IC2.9 (4A), JP3.2 (B), U2.11 (PD7)
- new net TTL_SPI_MOSI: IC2.7 (3A), JP6.2 (B), TP6.1, U2.15 (PB3)
- new net TTL_SPI_SCLK: IC2.3 (1A), JP4.2 (B), TP8.1, U2.17 (PB5)
- new net TTL_SS: IC2.5 (2A), JP5.2 (B), TP5.1, U2.14 (PB2)
- new net VCC: C14.1, C15.1, C16.1, JP2.2 (C), U2.18 (AVCC), U2.4 (VCC), U2.6 (VCC)
- no-connect marks 14 -> 24
Other:
- note added: "CL=(C1*C2)/(C1+C2) + Cstray\nCL = 20pF\nCstray = 5pF\nC1, C2 = 30pF\n"
- note added: "CL=(C1*C2)/(C1+C2) + Cstray\nCL = 9pF\nCstray = 5pF\nC1, C2 = 4pF\n"
- note added: "Cut if ATMEGA is running at 5v"
- note added: "Only needed if the ATMEGA is running at 5v"
- moved on the sheet: J3, R3, R6, R7
