File: hw/adbuino_v0p9p1/LevelShifter.sch (KiCad schematic (older format))
At the start: 3 parts, among them Q1 BSS138

Commit message: First round of routing completed
Parts:
- R8, R9: LCSC C17414 -> C25744
Changed lines of the file:
@@
 F 2 "Resistor_SMD:R_0402_1005Metric" H 2050 2200 50  0001 C CNN
 F 3 "~" H 2050 2200 50  0001 C CNN
-F 4 "C17414" V 2050 2200 50  0001 C CNN "LCSC"
+F 4 "C25744" V 2050 2200 50  0001 C CNN "LCSC"
 	1    2050 2200
 	1    0    0    -1
@@
 F 2 "Resistor_SMD:R_0402_1005Metric" H 2800 2200 50  0001 C CNN
 F 3 "~" H 2800 2200 50  0001 C CNN
-F 4 "C17414" V 2800 2200 50  0001 C CNN "LCSC"
+F 4 "C25744" V 2800 2200 50  0001 C CNN "LCSC"
 	1    2800 2200
 	1    0    0    -1
