File: hw/adbuino_v1p0/adbuino.kicad_pcb (KiCad board)
At the start: 2 copper layers, 25 x 50 mm, 52 parts, among them IC1 MAX3421EEHJ+, J1 Conn_01x06_Male, J2 U254-051N-4BH806, J3 USB_A, J4 Mini-DIN-4, J5 Mini-DIN-4, J6 ICSP Programmer, Q1 BSS138, Q2 BSS138, U1 AMS1117-3.3, U2 ATmega328P-AU, Y1 16MHz, Y2 12MHz

Commit message: Created version 1.0 of USB ADBuino
Parts:
- removed TP11, TP12, TP13: TestPoint_Small, TestPoint:TestPoint_Pad_D1.0mm
- added JP1: SolderJumper_3_Bridged12, Jumper:SolderJumper-3_P1.3mm_Bridged12_RoundedPad1.0x1.5mm, F.Cu at (40.4, 72.6)
- added JP2: SolderJumper_3_Bridged12, Jumper:SolderJumper-3_P1.3mm_Bridged12_RoundedPad1.0x1.5mm, F.Cu at (42.9, 72.6)
- added JP3: SolderJumper_3_Bridged12, Jumper:SolderJumper-3_P1.3mm_Bridged12_RoundedPad1.0x1.5mm, F.Cu at (32.0, 72.6)
- added JP4: SolderJumper_3_Bridged12, Jumper:SolderJumper-3_P1.3mm_Bridged12_RoundedPad1.0x1.5mm, F.Cu at (34.5, 72.6)
- added TP1: TestPoint_Small, TestPoint:TestPoint_THTPad_D1.0mm_Drill0.5mm, B.Cu at (47.8, 39.9)
- added TP2: TestPoint_Small, TestPoint:TestPoint_THTPad_D1.0mm_Drill0.5mm, B.Cu at (48.8, 41.7)
- added TP3: TestPoint_Small, TestPoint:TestPoint_THTPad_D1.0mm_Drill0.5mm, B.Cu at (46.7, 41.7)
- moved R8 7.90 mm to (38.6, 73.9), turned to 90 degrees
- moved R11 7.38 mm to (36.3, 71.9), turned to 270 degrees
- moved R10 3.88 mm to (36.3, 73.9), turned to 90 degrees
- moved R9 2.95 mm to (38.6, 71.9), turned to 270 degrees
- moved Q2 2.56 mm to (29.0, 70.9)
- moved R16 2.51 mm to (44.7, 43.7), turned to 45 degrees
- moved Q1 2.49 mm to (46.0, 70.9)
- moved R13 1.63 mm to (43.9, 42.9), turned to 45 degrees
- moved R2 1.54 mm to (42.7, 68.2), turned to 180 degrees
- moved R15 0.80 mm to (43.2, 42.2), turned to 45 degrees
- moved R14 0.57 mm to (42.4, 41.4), turned to 45 degrees
Connections:
- J2 pad 2: (no net) -> Net-(J2-Pad2)
- J2 pad 3: (no net) -> Net-(J2-Pad3)
- J2 pad 4: (no net) -> Net-(J2-Pad4)
- Q1 pad 2: ADB_DATA_LV -> Net-(JP1-Pad2)
- Q1 pad 3: ADB_1_DATA -> Net-(JP2-Pad2)
- Q2 pad 2: ADB_PWR_ON_LV -> Net-(JP3-Pad2)
- Q2 pad 3: ADB_1_PWR_ON -> Net-(JP4-Pad2)
Routing:
- net ATMEGA_SPI_MOSI: track 64.8 -> 43.1 mm, vias 5 -> 3
- net Net-(J2-Pad3): track 0.00 -> 15.0 mm, vias 0 -> 1
- net Net-(J2-Pad4): track 0.00 -> 14.6 mm, vias 0 -> 1
- net Net-(J2-Pad2): track 0.00 -> 12.8 mm, vias 0 -> 1
- net +3V3: track 118.3 -> 129.4 mm, vias 10 -> 12
- net ADB_1_5v: track 29.0 -> 18.3 mm
- net Net-(JP4-Pad2): track 0.00 -> 9.34 mm, vias 0 -> 2
- net Net-(JP1-Pad2): track 0.00 -> 9.25 mm, vias 0 -> 2
- net MAX3421_RESET: track 31.4 -> 23.2 mm
- net DEBUG_LED: track 29.8 -> 22.8 mm
- net ATMEGA_SPI_SCLK: track 55.9 -> 49.7 mm
- net GND: track 156.2 -> 162.0 mm, vias 13 -> 17
- net Net-(JP2-Pad2): track 0.00 -> 5.28 mm
- net ATMEGA_SS: track 33.9 -> 29.9 mm
- net ATMEGA_SPI_MISO: track 52.0 -> 48.5 mm
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Other:
- board text added: "3v"
- board text added: "5v"
- board text added: "JLCJLCJLCJLC"
