File: hw/adbuino_v1p1/LevelShifter.sch (KiCad schematic (older format))
At the start: 5 parts, among them Q1 BSS138

Commit message: Current version
Parts:
- Q1: LCSC C52895 -> C78284
Changed lines of the file:
@@
 F 2 "Package_TO_SOT_SMD:SOT-23" H 3250 2375 50  0001 L CIN
 F 3 "https://www.onsemi.com/pub/Collateral/BSS138-D.PDF" H 3050 2450 50  0001 L CNN
-F 4 "C52895" H 3050 2450 50  0001 C CNN "LCSC"
+F 4 "C78284" H 3050 2450 50  0001 C CNN "LCSC"
 	1    3050 2450
 	1    0    0    1
