File: hw/adbuino_v1p1/adbuino.kicad_pcb (KiCad board)
At the start: 2 copper layers, 25 x 50 mm, 58 parts, among them IC1 MAX3421EEHJ+, J1 Conn_01x06_Male, J2 U254-051N-4BH806, J3 USB_A, J4 Mini-DIN-4, J5 Mini-DIN-4, J6 ICSP Programmer, J7 Conn_01x02_Male, Q1 BSS138, Q2 BSS138, U1 AMS1117-3.3, U2 ATmega328P-AU, Y1 16MHz, Y2 12MHz

Commit message: Current version
Parts:
- added D4: LED_Small, LED_SMD:LED_0805_2012Metric, F.Cu at (26.1, 54.6)
- added H1: MountingHole, MountingHole:MountingHole_3.2mm_M3, F.Cu at (30.5, 46.0)
- added R18: 10k, Resistor_SMD:R_0402_1005Metric, F.Cu at (29.5, 64.3)
- moved J7 26.3 mm to (47.8, 39.1), turned to 270 degrees
- moved R17 23.4 mm to (47.8, 41.9), turned to 180 degrees
- moved C11 15.4 mm to (42.9, 38.6), turned to 90 degrees
- moved Y2 12.2 mm to (40.6, 38.4), turned to 90 degrees
- moved C10 11.2 mm to (38.1, 39.1)
- moved TP2 9.52 mm to (47.2, 32.3)
- moved TP1 9.20 mm to (48.8, 30.7)
- moved TP3 8.13 mm to (48.8, 33.8)
- moved R5 0.78 mm to (30.2, 40.4)
- moved R4 0.78 mm to (30.2, 41.4)
Connections:
- U2 pad 2: (no net) -> OPTION_SELECT
- U2 pad 24: OPTION_SELECT -> USB_STAT_LED
Routing:
- net GND: track 162.2 -> 200.5 mm, vias 15 -> 16
- net Net-(C10-Pad1): track 5.25 -> 21.9 mm, vias 0 -> 2
- net Net-(J2-Pad3): track 15.0 -> 3.00 mm, vias 1 -> 0
- net USB_STAT_LED: track 0.00 -> 11.8 mm
- net Net-(D4-Pad2): track 0.00 -> 11.4 mm, vias 0 -> 2
- net +3V3: track 134.5 -> 144.5 mm
- net Net-(J2-Pad4): track 14.6 -> 4.89 mm, vias 1 -> 0
- net Net-(J2-Pad2): track 12.8 -> 4.89 mm, vias 1 -> 0
- net Net-(C11-Pad1): track 8.01 -> 14.0 mm, vias 0 -> 2
- net OPTION_SELECT: track 23.3 -> 29.1 mm, vias 2 -> 1
- net ADB_DATA_LV: track 22.3 -> 21.3 mm
- net Net-(D1-Pad2): track 7.52 -> 8.33 mm
- net ADB_1_DATA: track 22.9 -> 23.6 mm, vias 3 -> 2
- net MAX3421_RESET: track 23.2 -> 23.8 mm
- net Net-(D2-Pad2): track 4.87 -> 5.38 mm
Other:
- board text added: "ADB"
- board text added: "Data"
- board text added: "USB"
- board text removed: "STAT"
