File: hw/adbuino_v1p1/adbuino.sch (KiCad schematic (older format))
At the start: 48 parts, among them IC1 MAX3421EEHJ+, J1 Conn_01x06_Male, J2 U254-051N-4BH806, J3 USB_A, J4 Mini-DIN-4, J5 Mini-DIN-4, J6 ICSP Programmer, J7 Conn_01x02_Male, U1 AMS1117-3.3, U2 ATmega328P-AU, Y1 16MHz, Y2 12MHz

Commit message: Current version
Parts:
- added D4: LED_Small, LED_SMD:LED_0805_2012Metric, symbol Device:LED_Small
- added H1: MountingHole, MountingHole:MountingHole_3.2mm_M3, symbol Mechanical:MountingHole
- added R18: 10k, Resistor_SMD:R_0402_1005Metric, symbol Device:R_Small
Connections:
- net GND: now also D4.1 (K)
- net OPTION_SELECT: now also U2.2 (PD4); no longer U2.24 (PC1)
- new net: D4.2 (A), R18.2
- new net USB_STAT_LED: R18.1, U2.24 (PC1)
- no-connect marks 26 -> 25
Other:
- moved on the sheet: D1, D2, D3, J7, R12, R17, R4, R5
